File: LPC114/$LPC114.sch (KiCad schematic (older format))
At the start: 52 parts, among them CON1 BARREL_JACK, IC1 LM1117, IC2 LM1117, P1 CONN_01X28, P2 JTAG, P3 CONN_01X28, P4 CONN_01X07, SW1 SW_PUSH, SW2 SPST, SW3 SW_PUSH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

Commit message: added final files
Other:
- moved on the sheet: C8, C9
Changed lines of the file:
@@
 L C C8
 U 1 1 55B85F50
-P 3950 4200
-F 0 "C8" H 4000 4300 50  0000 L CNN
-F 1 "0.1uF" H 3950 4100 50  0000 L CNN
-F 2 "" H 3988 4050 30  0000 C CNN
-F 3 "" H 3950 4200 60  0000 C CNN
-	1    3950 4200
+P 4450 4150
+F 0 "C8" H 4500 4250 50  0000 L CNN
+F 1 "0.1uF" H 4450 4050 50  0000 L CNN
+F 2 "" H 4488 4000 30  0000 C CNN
+F 3 "" H 4450 4150 60  0000 C CNN
+	1    4450 4150
 	1    0    0    -1
 $EndComp
@@
 L C C9
 U 1 1 55B86E1B
-P 4200 4200
-F 0 "C9" H 4250 4300 50  0000 L CNN
-F 1 "0.1uF" H 4200 4100 50  0000 L CNN
-F 2 "" H 4238 4050 30  0000 C CNN
-F 3 "" H 4200 4200 60  0000 C CNN
-	1    4200 4200
+P 4700 4150
+F 0 "C9" H 4750 4250 50  0000 L CNN
+F 1 "0.1uF" H 4700 4050 50  0000 L CNN
+F 2 "" H 4738 4000 30  0000 C CNN
+F 3 "" H 4700 4150 60  0000 C CNN
+	1    4700 4150
 	1    0    0    -1
 $EndComp
@@
 L +3.3VP #PWR02
 U 1 1 55B86FBF
-P 3950 3950
-F 0 "#PWR02" H 4000 3980 20  0001 C CNN
-F 1 "+3.3VP" H 3950 4040 30  0000 C CNN
-F 2 "" H 3950 3950 60  0000 C CNN
-F 3 "" H 3950 3950 60  0000 C CNN
-	1    3950 3950
+P 4450 3900
+F 0 "#PWR02" H 4500 3930 20  0001 C CNN
+F 1 "+3.3VP" H 4450 3990 30  0000 C CNN
+F 2 "" H 4450 3900 60  0000 C CNN
+F 3 "" H 4450 3900 60  0000 C CNN
+	1    4450 3900
 	1    0    0    -1
 $EndComp
@@
 L GND #PWR03
 U 1 1 55B8705E
-P 3950 4450
-F 0 "#PWR03" H 3950 4200 60  0001 C CNN
-F 1 "GND" H 3950 4300 60  0000 C CNN
-F 2 "" H 3950 4450 60  0000 C CNN
-F 3 "" H 3950 4450 60  0000 C CNN
-	1    3950 4450
+P 4450 4400
+F 0 "#PWR03" H 4450 4150 60  0001 C CNN
+F 1 "GND" H 4450 4250 60  0000 C CNN
+F 2 "" H 4450 4400 60  0000 C CNN
+F 3 "" H 4450 4400 60  0000 C CNN
+	1    4450 4400
 	1    0    0    -1
 $EndComp
@@
 Wire Wire Line
 	3600 900  3600 800
-Connection ~ 4200 4000
-Connection ~ 4200 4400
-Wire Wire Line
-	3950 3950 3950 4000
-Wire Wire Line
-	3950 4400 3950 4450
+Connection ~ 4700 3950
+Connection ~ 4700 4350
+Wire Wire Line
+	4450 3900 4450 3950
+Wire Wire Line
+	4450 4350 4450 4400
 Wire Wire Line
 	3400 3750 3600 3750
@@
 NoConn ~ 2300 3100
 Wire Wire Line
-	3950 4000 4200 4000
-Wire Wire Line
-	4200 4400 3950 4400
+	4450 3950 4700 3950
+Wire Wire Line
+	4700 4350 4450 4350
 $Comp
 L CONN_01X28 P1
