File: LPC114/LPC114.sch (KiCad schematic (older format))
At the start: 64 parts

Commit message: added 2nd step files
Parts:
- removed C?: C, symbol C
- removed CON?: USB-MINI-B, symbol USB-MINI-B
- removed D?: LED, symbol LED
- removed P? (x2): CONN_01X40, symbol CONN_01X40
- removed Q?: BC856, SOT-23, symbol BC856
- removed R? (x7): R, symbol R
- added P1, P3: CONN_01X30, symbol CONN_01X30
- C1, C3, C6: renamed from C?; value C -> 0.1uF
- D2: renamed from D?; value DIODE -> IN4148
- P2: renamed from P?; value CONN_02X10 -> JTAG
- R1: renamed from R?; value R -> 470E
- X2: renamed from X?; value CRYSTAL -> 3.768KHz
- gave numbers to parts that had none: 44
Connections:
- net +3.3VP: now also P3.2 (P2)
- net +5V: now also P1.2 (P2); no longer C12.1
- net GND: now also C12.1, R12.1, R13.1, R14.1, R15.1, P1.1 (P1), P3.1 (P1); no longer D4.2 (K), D5.2 (K), D6.2 (K), D7.2 (K)
- net ISP: now also U1.4 (PIO0_1/CLKOUT/CT32B0_MAT2), P1.4 (P4)
- net P2_0: now also D4.1 (A), P1.15 (P15), P3.11 (P11); no longer R12.2
- net P2_1: now also D5.1 (A), P1.16 (P16), P3.12 (P12); no longer R13.2
- net P2_10: now also P1.25 (P25)
- net P2_11: now also P1.26 (P26)
- net P2_2: now also D6.1 (A), P1.17 (P17), P3.13 (P13); no longer R14.2
- net P2_3: now also D7.1 (A), P1.18 (P18), P3.14 (P14); no longer R15.2
- net P2_6: now also P1.21 (P21)
- net P2_7: now also P1.22 (P22)
- net P2_8: now also P1.23 (P23)
- net P2_9: now also P1.24 (P24)
- net P3_0: now also P3.4 (P4)
- net P3_1: now also P3.5 (P5)
- net P3_2: now also P3.6 (P6)
- net P3_3: now also P3.7 (P7)
- net P3_4: now also P3.8 (P8)
- net RESET: now also P1.3 (P3), P3.3 (P3)
- net RXD: now also U1.46 (PIO1_6/RXD/CT32B0_MAT0), P3.23 (P23), P3.9 (P9)
- net SCL: now also P1.7 (P7), P3.15 (P15)
- net SDA: now also P1.8 (P8), P3.16 (P16)
- net SWCLK: now also P1.13 (P13)
- net SWDIO: now also P3.20 (P20)
- net SWO: now also P1.12 (P12)
- net TXD: now also U1.47 (PIO1_7/TXD/CT32B0_MAT1), P3.10 (P10), P3.24 (P24)
- net WAKEUP: now also U1.40 (PIO1_4/AD5/CT32B1_MAT3/WAKEUP), P3.21 (P21)
- net at U1.10 (PIO0_2/SSEL0/CT16B0_CAP0): now also P1.5 (P5)
- net at U1.14 (PIO0_3): now also P1.6 (P6)
- net at U1.17 (PIO1_9/CT16B1_MAT0): now also P3.26 (P26)
- net at U1.19 (PIO2_4): now also P1.19 (P19)
- net at U1.20 (PIO2_5): now also P1.20 (P20)
- net at U1.22 (PIO0_6/SCK0): now also P1.9 (P9)
- net at U1.23 (PIO0_7/~CTS~): now also P1.10 (P10)
- net at U1.27 (PIO0_8/MISO0/CT16B0_MAT0): now also P1.11 (P11)
- net at U1.30 (PIO1_10/AD6/CT16B1_MAT1): now also P3.27 (P27)
- net at U1.32 (PIO0_11/AD0/CT32B0_MAT3/R): now also P1.14 (P14)
- net at U1.33 (PIO1_0/AD1/CT32B1_CAP0/R): now also P3.17 (P17)
- net at U1.34 (PIO1_1/AD2/CT32B1_MAT0/R): now also P3.18 (P18)
- net at U1.35 (PIO1_2/AD3/CT32B1_MAT1/R): now also P3.19 (P19)
- net at U1.42 (PIO1_11/AD7): now also P3.28 (P28)
- net at U1.45 (PIO1_5/~RTS~/CT32B0_CAP0): now also P3.22 (P22)
- net at U1.9 (PIO1_8/CT16B1_CAP0): now also P3.25 (P25)
- new net: D4.2 (K), R12.2
- new net: D5.2 (K), R13.2
- new net: D6.2 (K), R14.2
- new net: D7.2 (K), R15.2
- no-connect marks 3 -> 10
Other:
- moved on the sheet: C12, D4, D5, D6, D7, R12, R13, R14, R15

Commit message: added final files
Parts:
- removed C10, C11: 0.1uF, symbol C
- removed P1, P3: CONN_01X30, symbol CONN_01X30
- added P1, P3: CONN_01X28, symbol CONN_01X28
- added P4: CONN_01X07, symbol CONN_01X07
Connections:
- net +3.3VP: now also P3.2 (P2)
- net +5V: now also P1.2 (P2), P4.3 (P3)
- net GND: now also BT1.1 (+), C13.2, P2.10 (P10), P2.12 (P12), P2.14 (P14), P2.16 (P16), P2.18 (P18), P2.20 (P20), P2.4 (P4), P2.6 (P6), P2.8 (P8), U2.4 (GND), P1.1 (P1), P3.1 (P1), P4.1 (P1)
- net ISP: now also P1.4 (P4)
- net P2_0: now also P1.15 (P15), P3.11 (P11)
- net P2_1: now also P1.16 (P16), P3.12 (P12)
- net P2_10: now also P1.25 (P25)
- net P2_11: now also P1.26 (P26)
- net P2_2: now also P1.17 (P17), P3.13 (P13)
- net P2_3: now also P1.18 (P18), P3.14 (P14)
- net P2_6: now also P1.21 (P21)
- net P2_7: now also P1.22 (P22)
- net P2_8: now also P1.23 (P23)
- net P2_9: now also P1.24 (P24)
- net P3_0: now also P3.4 (P4)
- net P3_1: now also P3.5 (P5)
- net P3_2: now also P3.6 (P6)
- net P3_3: now also P3.7 (P7)
- net P3_4: now also P3.8 (P8)
- net RESET: now also P1.3 (P3), P3.3 (P3), P4.7 (P7)
- net RXD: now also P3.23 (P23), P3.9 (P9), P4.4 (P4)
- net SCL: now also P1.7 (P7), P3.15 (P15)
- net SDA: now also P1.8 (P8), P3.16 (P16)
- net SWCLK: now also P1.13 (P13)
- net SWDIO: now also P3.20 (P20)
- net SWO: now also P1.12 (P12)
- net TXD: now also P3.10 (P10), P3.24 (P24), P4.5 (P5)
- net WAKEUP: now also P3.21 (P21)
- net at U1.10 (PIO0_2/SSEL0/CT16B0_CAP0): now also P1.5 (P5)
- net at U1.14 (PIO0_3): now also P1.6 (P6)
- net at U1.17 (PIO1_9/CT16B1_MAT0): now also P3.26 (P26)
- net U_SW: now reaches U1.19 (PIO2_4)
- net U_SW: now also R5.2, SW5.1, P1.19 (P19)
- net at U1.20 (PIO2_5): now also P1.20 (P20)
- net at U1.22 (PIO0_6/SCK0): now also P1.9 (P9)
- net at U1.23 (PIO0_7/~CTS~): now also P1.10 (P10)
- net at U1.27 (PIO0_8/MISO0/CT16B0_MAT0): now also P1.11 (P11)
- net at U1.30 (PIO1_10/AD6/CT16B1_MAT1): now also P3.27 (P27)
- net at U1.32 (PIO0_11/AD0/CT32B0_MAT3/R): now also P1.14 (P14)
- net at U1.33 (PIO1_0/AD1/CT32B1_CAP0/R): now also P3.17 (P17)
- net at U1.34 (PIO1_1/AD2/CT32B1_MAT0/R): now also P3.18 (P18)
- net at U1.35 (PIO1_2/AD3/CT32B1_MAT1/R): now also P3.19 (P19)
- net at U1.42 (PIO1_11/AD7): now also P3.28 (P28)
- net at U1.45 (PIO1_5/~RTS~/CT32B0_CAP0): now also P3.22 (P22)
- net at U1.9 (PIO1_8/CT16B1_CAP0): now also P3.25 (P25)
- net P3_5: no longer names the net of U1.21 (PIO3_5)
- no-connect marks 10 -> 9
Changed lines of the file:
@@
-$EndComp
-$Comp
-L C C10
-U 1 1 55B86E45
-P 4450 4200
-F 0 "C10" H 4500 4300 50  0000 L CNN
-F 1 "0.1uF" H 4450 4100 50  0000 L CNN
-F 2 "" H 4488 4050 30  0000 C CNN
-F 3 "" H 4450 4200 60  0000 C CNN
-	1    4450 4200
-	1    0    0    -1
-$EndComp
-$Comp
-L C C11
-U 1 1 55B86E6C
-P 4700 4200
-F 0 "C11" H 4750 4300 50  0000 L CNN
-F 1 "0.1uF" H 4700 4100 50  0000 L CNN
-F 2 "" H 4738 4050 30  0000 C CNN
-F 3 "" H 4700 4200 60  0000 C CNN
-	1    4700 4200
-	1    0    0    -1
 $EndComp
 $Comp
@@
 Wire Wire Line
 	3600 900  3600 800
-Wire Wire Line
-	3950 4000 4700 4000
 Connection ~ 4200 4000
-Connection ~ 4450 4000
-Wire Wire Line
-	3950 4400 4700 4400
 Connection ~ 4200 4400
-Connection ~ 4450 4400
 Wire Wire Line
 	3950 3950 3950 4000
@@
 Text GLabel 6150 1650 0    40   Input ~ 0
 P3_4
-Text GLabel 2250 3100 0    40   Input ~ 0
-P3_5
-Wire Wire Line
-	2250 3100 2300 3100
 Wire Wire Line
 	4700 1150 5850 1150
@@
 	9650 6350 10800 6350
 Wire Wire Line
-	9650 6350 9650 6000
+	9650 6000 9650 6400
 NoConn ~ 10250 5100
 $Comp
@@
 	5600 5400 5750 5400
 Wire Wire Line
-	5750 5400 5750 6200
+	5750 5400 5750 6250
 Wire Wire Line
 	5750 6200 5600 6200
@@
 	6150 1650 6200 1650
 NoConn ~ 1000 3650
-NoConn ~ 1000 3750
-NoConn ~ 1000 3850
-NoConn ~ 6200 3750
-NoConn ~ 6200 3850
 Text GLabel 4700 1750 2    40   Input ~ 0
 RXD
@@
 TXD
 NoConn ~ 2100 3800
-$Comp
-L CONN_01X30 P1
-U 1 1 55B99FDC
-P 800 2400
-F 0 "P1" H 800 3950 50  0000 C CNN
-F 1 "CONN_01X30" V 900 2400 50  0000 C CNN
-F 2 "" H 800 2400 60  0000 C CNN
-F 3 "" H 800 2400 60  0000 C CNN
-	1    800  2400
-	-1   0    0    -1
-$EndComp
-$Comp
-L CONN_01X30 P3
-U 1 1 55B9A04D
-P 6400 2400
-F 0 "P3" H 6400 3950 50  0000 C CNN
-F 1 "CONN_01X30" V 6500 2400 50  0000 C CNN
-F 2 "" H 6400 2400 60  0000 C CNN
-F 3 "" H 6400 2400 60  0000 C CNN
-	1    6400 2400
-	1    0    0    -1
-$EndComp
 Wire Wire Line
 	6950 5250 7000 5250
@@
 	10300 4400 10300 4450
 NoConn ~ 1000 3550
+$Comp
+L CONN_01X07 P4
+U 1 1 55BAF2C5
+P 8300 1900
+F 0 "P4" H 8300 2300 50  0000 C CNN
+F 1 "CONN_01X07" V 8400 1900 50  0000 C CNN
+F 2 "" H 8300 1900 60  0000 C CNN
+F 3 "" H 8300 1900 60  0000 C CNN
+	1    8300 1900
+	-1   0    0    -1
+$EndComp
+$Comp
+L GND #PWR028
+U 1 1 55BAF493
+P 9200 1600
+F 0 "#PWR028" H 9200 1350 60  0001 C CNN
+F 1 "GND" H 9200 1450 60  0000 C CNN
+F 2 "" H 9200 1600 60  0000 C CNN
+F 3 "" H 9200 1600 60  0000 C CNN
+	1    9200 1600
+	1    0    0    -1
+$EndComp
+Wire Wire Line
+	8500 1600 9200 1600
+$Comp
+L +5V #PWR029
+U 1 1 55BAFA86
+P 8750 1800
+F 0 "#PWR029" H 8750 1650 60  0001 C CNN
+F 1 "+5V" H 8750 1940 60  0000 C CNN
+F 2 "" H 8750 1800 60  0000 C CNN
+F 3 "" H 8750 1800 60  0000 C CNN
+	1    8750 1800
+	0    1    1    0
+$EndComp
+Wire Wire Line
+	8500 1800 8750 1800
+NoConn ~ 8500 1700
+Text GLabel 8500 1900 2    40   Input ~ 0
+RXD
+Text GLabel 8500 2000 2    40   Input ~ 0
+TXD
+NoConn ~ 8500 2100
+Text GLabel 8500 2200 2    40   Input ~ 0
+RESET
+NoConn ~ 2300 3100
+Wire Wire Line
+	3950 4000 4200 4000
+Wire Wire Line
+	4200 4400 3950 4400
+$Comp
+L CONN_01X28 P1
+U 1 1 55BB2DC7
+P 800 2300
+F 0 "P1" H 800 3750 50  0000 C CNN
+F 1 "CONN_01X28" V 900 2300 50  0000 C CNN
+F 2 "" H 800 2300 60  0000 C CNN
+F 3 "" H 800 2300 60  0000 C CNN
+	1    800  2300
+	-1   0    0    -1
+$EndComp
+$Comp
+L CONN_01X28 P3
+U 1 1 55BB34FB
+P 6400 2300
+F 0 "P3" H 6400 3750 50  0000 C CNN
+F 1 "CONN_01X28" V 6500 2300 50  0000 C CNN
+F 2 "" H 6400 2300 60  0000 C CNN
+F 3 "" H 6400 2300 60  0000 C CNN
+	1    6400 2300
+	1    0    0    -1
+$EndComp
+Text GLabel 3400 5700 2    40   Input ~ 0
+U_SW
+Text GLabel 1000 2750 2    40   Input ~ 0
+U_SW
+$Comp
+L GND #PWR?
+U 1 1 55BB5A0C
+P 9650 6400
+F 0 "#PWR?" H 9650 6150 60  0001 C CNN
+F 1 "GND" H 9650 6250 60  0000 C CNN
+F 2 "" H 9650 6400 60  0000 C CNN
+F 3 "" H 9650 6400 60  0000 C CNN
+	1    9650 6400
+	1    0    0    -1
+$EndComp
+Connection ~ 9650 6350
+$Comp
+L GND #PWR?
+U 1 1 55BC6C35
+P 5750 6250
+F 0 "#PWR?" H 5750 6000 60  0001 C CNN
+F 1 "GND" H 5750 6100 60  0000 C CNN
+F 2 "" H 5750 6250 60  0000 C CNN
+F 3 "" H 5750 6250 60  0000 C CNN
+	1    5750 6250
+	1    0    0    -1
+$EndComp
+Connection ~ 5750 6200
 $EndSCHEMATC
