File: LPC114/LPC114.kicad_pcb (KiCad board)
At the start: 2 copper layers, 93 x 51 mm, 53 parts, among them CON1 BARREL_JACK, IC1 LM1117, IC2 LM1117, P1 CONN_01X30, P2 JTAG, P3 CONN_01X30, SW1 SW_PUSH, SW2 SPST, SW3 SW_PUSH, SW4 SW_PUSH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

Commit message: added final files
Parts:
- removed C10, C11: 0.1uF, Capacitors_SMD:C_0603_HandSoldering
- added LOGO: , Logo:LOGO (2), B.Cu at (141.4, 63.9)
- added P4: CONN_01X07, ExploreEmbedded:USB_Shield, F.Cu at (140.2, 82.3)
- P1, P3: value CONN_01X30 -> CONN_01X28; footprint Pin_Headers:Pin_Header_Straight_1x30 -> Pin_Headers:Pin_Header_Straight_1x28
- R12, R13, R14, R15: moved to F.Cu
- moved C13 37.2 mm to (106.3, 88.9), turned to 90 degrees
- moved BT1 37.1 mm to (106.2, 93.0)
- moved C7 30.3 mm to (134.9, 67.3)
- moved C5 27.3 mm to (146.8, 67.3)
- moved IC1 16.2 mm to (133.9, 77.2), turned to 0 degrees
- moved IC2 16.1 mm to (133.9, 86.9), turned to 0 degrees
- moved C8 14.9 mm to (125.8, 74.8), turned to 315 degrees
- moved R17 14.4 mm to (132.7, 96.6), turned to 180 degrees
- moved R16 13.3 mm to (132.7, 94.4), turned to 180 degrees
- moved X2 11.6 mm to (145.2, 97.5)
- moved C12 9.80 mm to (135.2, 92.6), turned to 0 degrees
- moved D3 7.75 mm to (159.6, 104.8), turned to 0 degrees
- moved D2 7.00 mm to (156.8, 96.5)
- moved U2 6.31 mm to (139.6, 96.5), turned to 180 degrees
- moved R11 5.59 mm to (159.3, 102.5), turned to 180 degrees
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Connections:
- net P3_5 renamed Net-(U1-Pad21)
- BT1 pad 1: Net-(BT1-Pad1) -> GND
- C13 pad 2: Net-(BT1-Pad1) -> GND
- P1 pad 19: Net-(P1-Pad19) -> U_SW
- P2 pad 10: Net-(P2-Pad10) -> GND
- P2 pad 12: Net-(P2-Pad10) -> GND
- P2 pad 14: Net-(P2-Pad10) -> GND
- P2 pad 16: Net-(P2-Pad10) -> GND
- P2 pad 18: Net-(P2-Pad10) -> GND
- P2 pad 20: Net-(P2-Pad10) -> GND
- P2 pad 4: Net-(P2-Pad10) -> GND
- P2 pad 6: Net-(P2-Pad10) -> GND
- P2 pad 8: Net-(P2-Pad10) -> GND
- R5 pad 2: Net-(R5-Pad2) -> U_SW
- SW5 pad 1: Net-(R5-Pad2) -> U_SW
- U1 pad 19: Net-(P1-Pad19) -> U_SW
- U2 pad 4: Net-(BT1-Pad1) -> GND
Routing:
- net GND: track 0.00 -> 354.8 mm, vias 0 -> 13
- net +5V: track 0.00 -> 209.8 mm, vias 0 -> 4
- net +3.3VP: track 0.00 -> 204.8 mm, vias 0 -> 12
- net RESET: track 0.00 -> 153.8 mm, vias 0 -> 6
- net SDA: track 0.00 -> 132.4 mm, vias 0 -> 2
- net SCL: track 0.00 -> 126.3 mm, vias 0 -> 1
- net SWDIO: track 0.00 -> 121.9 mm, vias 0 -> 1
- net Net-(C5-Pad2): track 0.00 -> 115.1 mm, vias 0 -> 3
- net RXD: track 0.00 -> 111.7 mm, vias 0 -> 5
- net TXD: track 0.00 -> 109.3 mm, vias 0 -> 4
- net Net-(BT1-Pad2): track 0.00 -> 94.2 mm, vias 0 -> 2
- net P2_2: track 0.00 -> 91.1 mm, vias 0 -> 2
- net SWO: track 0.00 -> 87.3 mm, vias 0 -> 4
- net P3_2: track 0.00 -> 84.7 mm, vias 0 -> 3
- net ISP: track 0.00 -> 80.2 mm, vias 0 -> 3
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Other:
- board size 93 x 51 mm -> 90 x 51 mm
- net class Default: clearance 0.254 -> 0.1778
- rule trace_clearance: 0.254 -> 0.1778
- rule trace_min: 0.254 -> 0.2032
- board text added: "Explore LPC1114 Breakout"
- board text added: "ExploreEmbedded.com"
- board text added: "ISP"
- board text added: "RESET"
- board text added: "U_SW"
- board text added: "WAKEUP"

Commit message: gerber file added
Routing:
- added copper zone on F.Cu, net +3.3VP
- added copper zone on B.Cu, net GND
Other:
- board text added: "Explore Cortex M0 LPC1114"
- board text removed: "EploreEmbedded.com"
- board text removed: "Explore LPC1114 Breakout"

Commit message: Design errors
Other:
- board text added: "1. Gnd open 2. Connect RTS to ISP"
